File: electrical/smell_monitor_v1_1/smell_monitor_v1_1.kicad_sch (KiCad schematic)
At the start: 64 parts, among them J1 USB_C_16P, J10 JST-PH 2P fan, J2 1x05 female, J3 1x05 female, J4 1x05 female, J5 1x05 female, J6 1x06 female, J7 1x06 female, J8 1x06 female, J9 1x06 female, Q1 AO3400A, Q2 MMBT3904, SW1 MEASURE, SW2 BOOT, SW3 RESET, U1 ESP32-WROOM-32E, U2 ADS1115, U3 CH340C, U4 TCA9548A, U5 SHT31-DIS-B, U6 SSD1306-B, U7 AMS1117-3.3

Commit message: feat(electrical): generate, route and gate the v1.1 PCB
The routed board in git was not reproducible from anything committed. It is now
produced by a pipeline in which every stage refuses to do the dangerous thing:

- gen_pcb.py    placement only (outline, footprints, netclasses); refuses to
                overwrite a board that already carries copper without --force.
                The 8 sensing headers land exactly on interface.ANALOG_HEADERS /
                DIGITAL_HEADERS, i.e. exactly on the chamber wells.
- route_pcb.py  DSN -> FreeRouting (java -jar, -mp 12) -> SES; refuses to save
                unless 0 unconnected remain. Runs the router in the throwaway
                DSN/SES directory so it stops dropping en/freerouting.log in the
                repo root.
- export_fab.py the exact fab layer set (F/B Cu, mask, silkscreen, paste,
                Edge.Cuts) + Excellon drill + one CPL; deletes any stray layer
                left in fab/ by an older export.
- verify_pcb.py gate on the routed board: headers on the contract, outline,
                minimum track width, via stack, 0 unconnected, DRC clean.

Result: 847 segments, 102 vias, 0 unconnected, DRC 0 violations / 0 footprint
errors. The netclass track width goes 0.15 -> 0.30 mm because FreeRouting necks
to 75 %/50 % of nominal, which is what produced the earlier 109 track_width
violations; 0.30 is the smallest nominal that keeps every necked track at or
above the 0.15 mm board minimum.

fab/ is re-exported: 13 files instead of 29. The 16 cosmetic layers no board
shop can use (Adhesive, Courtyard, Fab, Margin, User_1..4, User_Comments,
User_Drawings, User_Eco1/2) and a 5 MB STEP are gone.

Also: verify_netlist.py now runs KiCad ERC itself (0 errors / 0 warnings)
instead of leaving "ERC clean" to a hand-run command that litters the working
tree; interface.py derives the two row Ys from the swapped geometry; board.py
fixes a cross-reference to a generator that never lived in tools/; bom.csv is
re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
Parts:
- BZ1: footprint Buzzer:Buzzer_12x9.5mm_D10.2mm -> Buzzer_Beeper:Buzzer_12x9.5RM7.6
- J10: footprint Connector_JST:JST_PH_B2B-PH-K-S_1x02_P2.00mm_Vertical -> Connector_JST:JST_PH_B2B-PH-K_1x02_P2.00mm_Vertical
- U5: footprint Package_DFN_QFN:DFN-8-1EP_2.5x2.5mm_P0.5mm_EP1.4x1.4mm -> Sensor_Humidity:Sensirion_DFN-8-1EP_2.5x2.5mm_P0.5mm_EP1.1x1.7mm
Other:
- note added: "1. +3V3 is generated by U7 (AMS1117CD-3.3) from the USB-C +5V rail; every IC has a 100nF decoupling cap at its supply pin."
- note added: "2. ANALOG SLOTS J2..J5 = 1:+5V 2:GND 3:AO 4:DO 5:3V3 (MQ-type module seats on pins 1-4)."
- note added: "3. DIGITAL SLOTS J6..J9 = 1:3V3 2:GND 3:SDA 4:SCL 5:INT 6:CTRL (each slot is one TCA9548A channel)."
- note added: "4. I2C ADDRESSES ADS1115 0x48 TCA9548A 0x70 SHT31 0x44 OLED 0x3C."
- note added: "5. S1 = MEASURE (start a sniff cycle) S2 = BOOT S3 = RESET. Manual flashing, no auto-reset transistors."
- note added: "6. Connectivity is carried by net-name labels; the authoritative pin/net model is electrical/board.py (validated, ERC-clean)."
- note added: "7. NC = not connected (no-connect flag placed). All dimensions mm; passives 0603 unless noted."
- note added: "ANALOG INPUT (ADS1115)"
- note added: "ANALOG SLOTS"
- note added: "DIGITAL SLOTS"
- note added: "I2C MULTIPLEXER (TCA9548A)"
- note added: "MICROCONTROLLER"
- note added: "NOTES"
- note added: "OUTPUTS"
- note added: "POWER SUPPLY"
- note added: "SENSOR / DISPLAY"
- note added: "USB  UART BRIDGE"
- company: (none) -> OpenSmell
- title: (none) -> OpenSmell v1.1   e-nose sensing platform (sheet 1 of 1)
